Commit message: Redesigned car
Car base is redesigned, add controller for left steering. Added
lidar in the car.

File: car_assem/urdf/car_assem.urdf (robot description, URDF)
Before this commit: robot car_assem, 8 links, 7 joints
Links:
- added link base_laser, mass 0.15717; collision mesh filename=package://car_assem/meshes/ydlidar.dae; visual mesh filename=package://car_assem/meshes/ydlidar.dae
- added link laser_frame, mass 0.25482
Joints:
- added joint laser_joint: type fixed, parent base_laser, child laser_frame, origin xyz=0 0 0.03172 rpy=0 0 0, axis 0 0 0
- added joint lidarGlue: type fixed, parent base_link, child base_laser, origin xyz=0 0 0 rpy=0 0 0
- joint back_left_wheel: origin xyz=0.60728 0.42837 1.0349 rpy=2.7212 -1.5708 0 -> xyz=-0.18569 0.254 -0.0889 rpy=1.9912 0 1.5708
- joint back_right_wheel: origin xyz=0.62095 0.42207 0.45072 rpy=1.2833 1.5708 0 -> xyz=-0.18569 -0.254 -0.0889 rpy=2.8541 0 -1.5708
- joint dummy_joint: origin xyz=0 0 0 rpy=1.5 0 0 -> xyz=0 0 0 rpy=0 0 0
- joint front_left_steering: origin xyz=0.091551 0.41654 0.92953 rpy=0 -1.5464 0 -> xyz=0.33413 0.14861 -0.0254 rpy=1.5708 0 1.5952
- joint front_left_wheel: origin xyz=0.084724 0.020158 -0.0087955 rpy=-1.0749 0 0 -> xyz=0.084724 -0.0508 0 rpy=-1.0749 0 0
- joint front_right_steering: origin xyz=0.091551 0.41654 0.6323 rpy=3.1416 1.548 3.1416 -> xyz=0.33413 -0.14861 -0.0254 rpy=1.5708 0 -1.548
- joint front_right_wheel: origin xyz=0.084938 0.021602 -0.0078446 rpy=-0.90183 0 0 -> xyz=0.084938 -0.0508 0 rpy=-0.90183 0 0
